Commit message: pick and place

File: src/ur5/urdf/ur5.urdf.xacro (robot description, xacro)
@@ -48,70 +48,64 @@
   <!--     xyz_offset="0.4 0.2 0.8" -->
   <!--     rpy_offset="3.14 0 1.57" /> -->
-  <joint name="camera_joint" type="fixed">
-    <parent link="base_link"/>
-    <child link="camera_link"/>
-    <origin xyz="0.4 0 1.0" rpy="0 1.57 0"/>
-  </joint>
-  <link name="camera_link">
-    <visual>
-      <geometry>
-	<box size="0.015 0.130 0.0222"/>
-      </geometry>
-    </visual>
-    <collision>
-      <geometry>
-	<box size="0.015 0.130 0.0222"/>
-      </geometry>
-    </collision>
-    <inertial>
-      <mass value="0.035"/>
-      <inertia ixx="1e-6" ixy="0" ixz="0" iyy="1e-6" iyz="0" izz="1e-6"/>
-      <origin xyz="0 0 0" rpy="0 0 0"/>
-    </inertial>
-  </link>
-  <gazebo reference="camera_link">
-    <sensor name="depth_camera" type="camera">
-      <update_rate>5.0</update_rate>
-      <always_on>true</always_on>
-      <visualize>true</visualize>
-      <topic>cam_1/image</topic>
-      <camera>
-	<horizontal_fov>1.4</horizontal_fov>
-	<image>
-          <width>640</width>
-          <height>480</height>
-          <format>R8G8B8</format>
-	</image>
-	<clip>
-          <near>0.05</near>
-          <far>3</far>
-	</clip>
-      </camera>
-    </sensor>
-    <sensor name="depth_camera_depth" type="depth">
-      <update_rate>5.0</update_rate>
-      <always_on>true</always_on>
-      <visualize>true</visualize>
-      <topic>depth_camera/depth_image</topic>
-      <camera>
-	<horizontal_fov>1.047198</horizontal_fov>
-	<image>
-          <width>640</width>
-          <height>480</height>
-          <format>R8G8B8</format>
-	</image>
-	<clip>
-          <near>0.05</near>
-          <far>3</far>
-	</clip>
-      </camera>
-    </sensor>
-  </gazebo>
-  <gazebo>
-    <plugin
-	filename="gz-sim-sensors-system"
-	name="gz::sim::systems::Sensors">
-      <render_engine>ogre2</render_engine>
-    </plugin>
-  </gazebo>
+  <!-- <joint name="camera_joint" type="fixed"> -->
+  <!--   <parent link="world"/> -->
+  <!--   <child link="camera_link"/> -->
+  <!--   <origin xyz="0.4 0 1.0" rpy="0 1.57 0"/> -->
+  <!-- </joint> -->
+  <!-- <link name="camera_link"> -->
+  <!--   <visual> -->
+  <!--     <geometry> -->
+  <!-- 	<box size="0.015 0.130 0.0222"/> -->
+  <!--     </geometry> -->
+  <!--   </visual> -->
+  <!--   <collision> -->
+  <!--     <geometry> -->
+  <!-- 	<box size="0.015 0.130 0.0222"/> -->
+  <!--     </geometry> -->
+  <!--   </collision> -->
+  <!--   <inertial> -->
+  <!--     <mass value="0.035"/> -->
+  <!--     <inertia ixx="1e-6" ixy="0" ixz="0" iyy="1e-6" iyz="0" izz="1e-6"/> -->
+  <!--     <origin xyz="0 0 0" rpy="0 0 0"/> -->
+  <!--   </inertial> -->
+  <!-- </link> -->
+  <!-- <gazebo reference="camera_link"> -->
+  <!--   <sensor name="depth_camera" type="rgbd_camera"> -->
+  <!--     <always_on>true</always_on> -->
+  <!--     <visualize>true</visualize> -->
+  <!--     <update_rate>5.0</update_rate> -->
+  <!--     <topic>depth_camera</topic> -->
+  <!--     <camera> -->
+  <!-- 	<horizontal_fov>1.047198</horizontal_fov> -->
+  <!-- 	<image> -->
+  <!-- 	  <width>640</width> -->
+  <!-- 	  <height>480</height> -->
+  <!-- 	</image> -->
+  <!-- 	<clip> -->
+  <!-- 	  <near>0.05</near> -->
+  <!-- 	  <far>3</far> -->
+  <!-- 	</clip> -->
+  <!--     </camera> -->
+  <!--     <baseline>0.2</baseline> -->
+  <!--     <pointCloudCutoff>0.5</pointCloudCutoff> -->
+  <!--     <pointCloudCutoffMax>3.0</pointCloudCutoffMax> -->
+  <!--     <distortionK1>0</distortionK1> -->
+  <!--     <distortionK2>0</distortionK2> -->
+  <!--     <distortionK3>0</distortionK3> -->
+  <!--     <distortionT1>0</distortionT1> -->
+  <!--     <distortionT2>0</distortionT2> -->
+  <!--     <CxPrime>0</CxPrime> -->
+  <!--     <Cx>0</Cx> -->
+  <!--     <Cy>0</Cy> -->
+  <!--     <focalLength>0</focalLength> -->
+  <!--     <hackBaseline>0</hackBaseline> -->
+  <!--   </sensor> -->
+  <!-- </gazebo> -->
+  <!-- <gazebo> -->
+  <!--   <plugin -->
+  <!-- 	filename="gz-sim-sensors-system" -->
+  <!-- 	name="gz::sim::systems::Sensors"> -->
+  <!--     <render_engine>ogre2</render_engine> -->
+  <!--   </plugin> -->
+  <!-- </gazebo> -->
 </robot>
